File: electronics/MyBikesGotLED.sch (KiCad schematic (older format))
At the start: 41 parts, among them J1 Battery, J2 WS2812, J3 Serial, J4 Battery_Test_Points, J5 Conn_01x04, Q1 FS8205, SW2 ON/OFF, U2 SN74AHCT125, U3 FS312F-G, U4 MT3608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

Commit message: Changed switch, finished laying out PCB.
Parts:
- added Q2: JSM2302, Package_TO_SOT_SMD:SOT-23, symbol Transistor_FET:DMN2041L
- added R18: R10K, Resistor_SMD:R_0603_1608Metric_Pad0.98x0.95mm_HandSolder, symbol Device:R_Small
- added R6: 100K, Resistor_SMD:R_0603_1608Metric_Pad0.98x0.95mm_HandSolder, symbol Device:R_Small
- J2: footprint Connector_PinHeader_2.54mm:PinHeader_1x03_P2.54mm_Vertical -> Connector_PinHeader_2.54mm:PinHeader_1x03_P2.54mm_Horizontal
- R12: value 10K -> R10K
- SW2: footprint (none) -> Button_Switch_THT:SW_CuK_OS102011MA1QN1_SPDT_Angled; Farnell (none) -> 1201431; Farnell Price/Stock (none) -> https://uk.farnell.com/c-k-components/os102011ma1qn1/switch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
- gave numbers to parts that had none: 2
Connections:
- net +BATT: now also C3.1, F1.2, JP2.1, L1.1, U4.5 (IN), R18.1; no longer JP1.1, SW2.1 (A)
- net -BATT: now also JP1.1, Q2.2 (S), R6.2; no longer C1.2, Q1.3 (S2), U3.6 (GND)
- net GND: now also J2.1 (Pin_1); no longer J2.3 (Pin_3)
- net at 5V_T1.1 (Pin_1), C5.1, C7.1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: now also J2.3 (Pin_3); no longer J2.1 (Pin_1)
- net at SW2.3 (C): now also Q2.1 (G), R6.1
- new net: C1.2, JP1.2, Q1.3 (S2), Q2.3 (D), U3.6 (GND)
- new net: R18.2, SW2.2 (B)
Other:
- moved on the sheet: C1, JP1, Q1, R11, R5, SW2, U3

Commit message: Change cap part number to one that's in stock.
Parts:
- C4: LCSC C28504 -> C342632; LCSC Price/Stock https://www.lcsc.com/product-detail/Multilayer-Ceramic-Capacitors-MLCC-SMD-SMT_FH_1812X226K250NT_22uF-226-10-25V_C28504.html -> https://www.lcsc.com/product-detail/Multilayer-Ceramic-Capacitors-MLCC-SMD-SMT_TDK-C4532X7R1C226MT000N_C342632.html
Changed lines of the file:
@@
 F 2 "Capacitor_SMD:C_1812_4532Metric_Pad1.57x3.40mm_HandSolder" H 5500 2900 50  0001 C CNN
 F 3 "~" H 5500 2900 50  0001 C CNN
-F 4 "C28504" H 5500 2900 50  0001 C CNN "LCSC"
-F 5 "https://www.lcsc.com/product-detail/Multilayer-Ceramic-Capacitors-MLCC-SMD-SMT_FH_1812X226K250NT_22uF-226-10-25V_C28504.html" H 5500 2900 50  0001 C CNN "LCSC Price/Stock"
+F 4 "C342632" H 5500 2900 50  0001 C CNN "LCSC"
+F 5 "https://www.lcsc.com/product-detail/Multilayer-Ceramic-Capacitors-MLCC-SMD-SMT_TDK-C4532X7R1C226MT000N_C342632.html" H 5500 2900 50  0001 C CNN "LCSC Price/Stock"
 	1    5500 2900
 	1    0    0    -1
